Commit message: fixed physics loop synchronization issues and added localization

File: workspace/src/robot_description/urdf/full_robot.xacro (robot description, xacro)
@@ -51,4 +51,17 @@
     <origin xyz="0 0 0.26" rpy="0 0 0"/>
   </joint>
+  <!-- frames for the LiDAR -->
+  <link name="front_lidar_frame"/>
+  <joint name="front_lidar_joint" type="fixed">
+    <parent link="base_link"/>
+    <child link="front_lidar_frame"/>
+    <origin xyz="0 0.4 0.2" rpy="0 0 1.57079632679"/>
+  </joint>
+  <link name="back_lidar_frame"/>
+  <joint name="back_lidar_joint" type="fixed">
+    <parent link="base_link"/>
+    <child link="back_lidar_frame"/>
+    <origin xyz="0 -0.4 0.2" rpy="0 0 -1.57079632679"/>
+  </joint>
   <!-- Four wheels from wheel.xacro.
        Positions are copied from robot.xml. -->

Commit message: added navigation stack (still not working)

File: workspace/src/robot_description/urdf/full_robot.xacro (robot description, xacro)
@@ -64,4 +64,12 @@
     <origin xyz="0 -0.4 0.2" rpy="0 0 -1.57079632679"/>
   </joint>
+  <!-- Front camera pose matches robot.xml's robot_camera.  The pi rotation
+       about X converts MuJoCo's camera convention to a ROS optical frame. -->
+  <link name="front_camera_frame"/>
+  <joint name="front_camera_joint" type="fixed">
+    <parent link="base_link"/>
+    <child link="front_camera_frame"/>
+    <origin xyz="0 0.51 0.22" rpy="-1.57079632679 0 -0.42760566673861"/>
+  </joint>
   <!-- Four wheels from wheel.xacro.
        Positions are copied from robot.xml. -->

File: workspace/src/robot_description/urdf/mujoco_config.xacro (robot description, xacro)
@@ -3,4 +3,5 @@
   <xacro:arg name="write_frequency" default="100"/>
   <xacro:arg name="physics_sync_safety_interval" default="0.002"/>
+  <xacro:arg name="extra_wait_time" default="0"/>
   <xacro:macro name="mujoco_ros2_control_config" params="">
   <ros2_control name="MujocoSystem" type="system">
@@ -12,5 +13,8 @@
         <param name="initial_keyframe">robot_above_floor</param>
         <param name="write_frequency">$(arg write_frequency)</param>
+        <!-- All MuJoCo camera streams are rendered and published at this rate. -->
+        <param name="camera_publish_rate">0.5</param>
         <param name="physics_sync_safety_interval">$(arg physics_sync_safety_interval)</param>
+        <param name="extra_wait_time">$(arg extra_wait_time)</param>
       </hardware>
       <!-- Four Wheel Joints -->
@@ -115,4 +119,11 @@
         <state_interface name="linear_acceleration.z"/>
       </sensor>
+      <!-- Front-facing MuJoCo camera (robot.xml: robot_camera). -->
+      <sensor name="robot_camera">
+        <param name="frame_name">front_camera_frame</param>
+        <param name="info_topic">/front_camera/depth/camera_info</param>
+        <param name="image_topic">/front_camera/image_raw</param>
+        <param name="depth_topic">/front_camera/depth/image_raw</param>
+      </sensor>
     </ros2_control>
   </xacro:macro>

Commit message: fixed orientation mismatch between mujoco and odometry

File: workspace/src/robot_description/urdf/full_robot.xacro (robot description, xacro)
@@ -10,6 +10,4 @@
     <color rgba="0.45 0.45 0.45 1.0"/>
   </material>
-  <!-- Root/world link -->
-  <link name="world"/>
   <!-- Base/chassis box.
        This is the main base link of the full robot. -->
@@ -44,11 +42,4 @@
     </collision>
   </link>
-  <!-- In MuJoCo, chassis is at pos="0 0 0.26".
-       For RViz/URDF visualization we fix it to world. -->
-  <joint name="world_to_base" type="fixed">
-    <parent link="world"/>
-    <child link="base_link"/>
-    <origin xyz="0 0 0.26" rpy="0 0 0"/>
-  </joint>
   <!-- frames for the LiDAR -->
   <link name="front_lidar_frame"/>

File: workspace/src/robot_description/urdf/mujoco_config.xacro (robot description, xacro)
@@ -11,5 +11,4 @@
         <param name="sim_speed_factor">0.5</param>
         <param name="headless">true</param>
-        <param name="initial_keyframe">robot_above_floor</param>
         <param name="write_frequency">$(arg write_frequency)</param>
         <!-- All MuJoCo camera streams are rendered and published at this rate. -->

Commit message: fixed orientation mismatch between mujoco and odometry 1

File: workspace/src/robot_description/urdf/full_robot.xacro (robot description, xacro)
@@ -15,5 +15,5 @@
     <inertial>
       <!-- MuJoCo chassis box:
-           size="0.40 0.5 0.05" means full size 0.80 x 1.00 x 0.10
+           size="0.5 0.40 0.05" means full size 1.00 x 0.80 x 0.10
            mass="10"
       -->
@@ -21,8 +21,8 @@
       <mass value="10.0"/>
       <inertia
-        ixx="0.842"
+        ixx="0.542"
         ixy="0.0"
         ixz="0.0"
-        iyy="0.542"
+        iyy="0.842"
         iyz="0.0"
         izz="1.367"/>
@@ -31,5 +31,5 @@
       <origin xyz="0 0 0.14" rpy="0 0 0"/>
       <geometry>
-        <box size="0.80 1.00 0.10"/>
+        <box size="1.00 0.80 0.10"/>
       </geometry>
       <material name="chassis_gray"/>
@@ -38,5 +38,5 @@
       <origin xyz="0 0 0.14" rpy="0 0 0"/>
       <geometry>
-        <box size="0.80 1.00 0.10"/>
+        <box size="1.00 0.80 0.10"/>
       </geometry>
     </collision>
@@ -63,25 +63,24 @@
     <origin xyz="0 0.51 0.22" rpy="-1.57079632679 0 -0.42760566673861"/>
   </joint>
-  <!-- Four wheels from wheel.xacro.
-       Positions are copied from robot.xml. -->
+  <!-- Match the MuJoCo chassis frame exactly: +Y is front and +X is left. -->
   <xacro:mecanum_wheel
     prefix="fr"
     parent="base_link"
-    xyz="0.25 -0.35 -0.1"
+    xyz="0.35 0.25 -0.1"
     rpy="0 0 -1.57079632679"/>
   <xacro:mecanum_wheel
     prefix="fl"
     parent="base_link"
-    xyz="0.25 0.35 -0.1"
+    xyz="-0.35 0.25 -0.1"
     rpy="0 0 -1.57079632679"/>
   <xacro:mecanum_wheel
     prefix="rr"
     parent="base_link"
-    xyz="-0.25 -0.35 -0.1"
+    xyz="0.35 -0.25 -0.1"
     rpy="0 0 -1.57079632679"/>
   <xacro:mecanum_wheel
     prefix="rl"
     parent="base_link"
-    xyz="-0.25 0.35 -0.1"
+    xyz="-0.35 -0.25 -0.1"
     rpy="0 0 -1.57079632679"/>
   <!-- Attach the arm rigidly to the mobile base. -->

Commit message: configured navigation stack

File: workspace/src/robot_description/urdf/full_robot.xacro (robot description, xacro)
@@ -47,5 +47,5 @@
     <parent link="base_link"/>
     <child link="front_lidar_frame"/>
-    <origin xyz="0 0.4 0.2" rpy="0 0 1.57079632679"/>
+    <origin xyz="0.4 0 0.2" rpy="0 0 0"/>
   </joint>
   <link name="back_lidar_frame"/>
@@ -53,35 +53,36 @@
     <parent link="base_link"/>
     <child link="back_lidar_frame"/>
-    <origin xyz="0 -0.4 0.2" rpy="0 0 -1.57079632679"/>
+    <origin xyz="-0.4 0 0.2" rpy="0 0 3.1415926535"/>
   </joint>
-  <!-- Front camera pose matches robot.xml's robot_camera.  The pi rotation
-       about X converts MuJoCo's camera convention to a ROS optical frame. -->
+  <!-- ROS optical frame matching robot.xml's forward-facing camera:
+       +X right, +Y down, and +Z forward along the chassis +X axis. -->
   <link name="front_camera_frame"/>
   <joint name="front_camera_joint" type="fixed">
     <parent link="base_link"/>
     <child link="front_camera_frame"/>
-    <origin xyz="0 0.51 0.22" rpy="-1.57079632679 0 -0.42760566673861"/>
+    <origin xyz="0.51 0 0.22"
+            rpy="-1.57079632679 0 -1.57079632679"/>
   </joint>
-  <!-- Match the MuJoCo chassis frame exactly: +Y is front and +X is left. -->
+  <!-- Match the MuJoCo chassis frame exactly: +X is front and +Y is left. -->
+  <xacro:mecanum_wheel
+    prefix="fl"
+    parent="base_link"
+    xyz="0.35 0.25 -0.1"
+    rpy="0 0 0"/>
+  <xacro:mecanum_wheel
+    prefix="rl"
+    parent="base_link"
+    xyz="-0.35 0.25 -0.1"
+    rpy="0 0 0"/>
   <xacro:mecanum_wheel
     prefix="fr"
     parent="base_link"
-    xyz="0.35 0.25 -0.1"
-    rpy="0 0 -1.57079632679"/>
-  <xacro:mecanum_wheel
-    prefix="fl"
-    parent="base_link"
-    xyz="-0.35 0.25 -0.1"
-    rpy="0 0 -1.57079632679"/>
+    xyz="0.35 -0.25 -0.1"
+    rpy="0 0 0"/>
   <xacro:mecanum_wheel
     prefix="rr"
     parent="base_link"
-    xyz="0.35 -0.25 -0.1"
-    rpy="0 0 -1.57079632679"/>
-  <xacro:mecanum_wheel
-    prefix="rl"
-    parent="base_link"
     xyz="-0.35 -0.25 -0.1"
-    rpy="0 0 -1.57079632679"/>
+    rpy="0 0 0"/>
   <!-- Attach the arm rigidly to the mobile base. -->
   <link name="arm_mount_link"/>
@@ -91,4 +92,7 @@
     <origin xyz="0 0 0.19" rpy="0 0 0"/>
   </joint>
-  <xacro:mujoco_ros2_control_config/>
+  <xacro:mujoco_ros2_control_config
+    write_frequency="$(arg write_frequency)"
+    physics_sync_safety_interval="$(arg physics_sync_safety_interval)"
+    extra_wait_time="$(arg extra_wait_time)"/>
 </robot>

File: workspace/src/robot_description/urdf/mujoco_config.xacro (robot description, xacro)
@@ -4,6 +4,7 @@
   <xacro:arg name="physics_sync_safety_interval" default="0.002"/>
   <xacro:arg name="extra_wait_time" default="0"/>
-  <xacro:macro name="mujoco_ros2_control_config" params="">
-  <ros2_control name="MujocoSystem" type="system">
+  <xacro:macro name="mujoco_ros2_control_config"
+               params="write_frequency physics_sync_safety_interval extra_wait_time">
+    <ros2_control name="MujocoSystem" type="system">
       <hardware>
         <plugin>mujoco_ros2_control/MujocoSystemInterface</plugin>
@@ -11,9 +12,9 @@
         <param name="sim_speed_factor">0.5</param>
         <param name="headless">true</param>
-        <param name="write_frequency">$(arg write_frequency)</param>
+        <param name="write_frequency">100</param>
+        <param name="physics_sync_safety_interval">0</param>
+        <param name="extra_wait_time">1</param>
         <!-- All MuJoCo camera streams are rendered and published at this rate. -->
         <param name="camera_publish_rate">1.0</param>
-        <param name="physics_sync_safety_interval">$(arg physics_sync_safety_interval)</param>
-        <param name="extra_wait_time">$(arg extra_wait_time)</param>
       </hardware>
       <!-- Four Wheel Joints -->

File: workspace/src/robot_description/urdf/wheel.xacro (robot description, xacro)
@@ -4,5 +4,6 @@
     <link name="${prefix}_wheel_link">
       <inertial>
-        <origin xyz="0 0 0" rpy="0 0 0"/>
+        <!-- Match the MJCF wheel body's inertial quaternion (90 deg about Z). -->
+        <origin xyz="0 0 0" rpy="0 0 1.57079632679"/>
         <mass value="6.5"/>
         <inertia

Commit message: fixed moveit config and URDF mismatches and added food items teleportation

File: workspace/src/robot_description/urdf/full_robot.xacro (robot description, xacro)
@@ -11,5 +11,12 @@
   </material>
   <!-- Base/chassis box.
-       This is the main base link of the full robot. -->
+       This is the main base link of the full robot.
+       base_link is the planar odometry frame: the EKF/AMCL stack publishes
+       map->odom->base_link with z=0 (two_d_mode). MuJoCo, however, spawns the
+       chassis body 0.26 m above the ground (robot.xml: chassis pos="0 0 0.26").
+       To keep the URDF/planning model at the true physical height while base_link
+       stays on the ground, every base_link child offset below includes that
+       0.26 m chassis height (e.g. chassis box 0.14 -> 0.40, wheels -0.1 -> 0.16,
+       arm mount 0.19 -> 0.45). -->
   <link name="base_link">
     <inertial>
@@ -18,5 +25,5 @@
            mass="10"
       -->
-      <origin xyz="0 0 0.14" rpy="0 0 0"/>
+      <origin xyz="0 0 0.40" rpy="0 0 0"/>
       <mass value="10.0"/>
       <inertia
@@ -29,5 +36,5 @@
     </inertial>
     <visual>
-      <origin xyz="0 0 0.14" rpy="0 0 0"/>
+      <origin xyz="0 0 0.40" rpy="0 0 0"/>
       <geometry>
         <box size="1.00 0.80 0.10"/>
@@ -36,5 +43,5 @@
     </visual>
     <collision>
-      <origin xyz="0 0 0.14" rpy="0 0 0"/>
+      <origin xyz="0 0 0.40" rpy="0 0 0"/>
       <geometry>
         <box size="1.00 0.80 0.10"/>
@@ -47,5 +54,5 @@
     <parent link="base_link"/>
     <child link="front_lidar_frame"/>
-    <origin xyz="0.4 0 0.2" rpy="0 0 0"/>
+    <origin xyz="0.4 0 0.46" rpy="0 0 0"/>
   </joint>
   <link name="back_lidar_frame"/>
@@ -53,5 +60,5 @@
     <parent link="base_link"/>
     <child link="back_lidar_frame"/>
-    <origin xyz="-0.4 0 0.2" rpy="0 0 3.1415926535"/>
+    <origin xyz="-0.4 0 0.46" rpy="0 0 3.1415926535"/>
   </joint>
   <!-- ROS optical frame matching robot.xml's forward-facing camera:
@@ -61,5 +68,5 @@
     <parent link="base_link"/>
     <child link="front_camera_frame"/>
-    <origin xyz="0.51 0 0.22"
+    <origin xyz="0.51 0 0.48"
             rpy="-1.57079632679 0 -1.57079632679"/>
   </joint>
@@ -68,20 +75,20 @@
     prefix="fl"
     parent="base_link"
-    xyz="0.35 0.25 -0.1"
+    xyz="0.35 0.25 0.16"
     rpy="0 0 0"/>
   <xacro:mecanum_wheel
     prefix="rl"
     parent="base_link"
-    xyz="-0.35 0.25 -0.1"
+    xyz="-0.35 0.25 0.16"
     rpy="0 0 0"/>
   <xacro:mecanum_wheel
     prefix="fr"
     parent="base_link"
-    xyz="0.35 -0.25 -0.1"
+    xyz="0.35 -0.25 0.16"
     rpy="0 0 0"/>
   <xacro:mecanum_wheel
     prefix="rr"
     parent="base_link"
-    xyz="-0.35 -0.25 -0.1"
+    xyz="-0.35 -0.25 0.16"
     rpy="0 0 0"/>
   <!-- Attach the arm rigidly to the mobile base. -->
@@ -90,5 +97,9 @@
     <parent link="base_link"/>
     <child link="arm_mount_link"/>
-    <origin xyz="0 0 0.19" rpy="0 0 0"/>
+    <!-- MuJoCo's arm_base body (mounted_arm.xml) is mounted with quat="0 0 0 -1",
+         a 180 degree yaw relative to its parent body. Match it here so the URDF
+         kinematic chain agrees with the physical mount orientation.
+         z = 0.26 (chassis height) + 0.19 (chassis top to arm base) = 0.45. -->
+    <origin xyz="0 0 0.45" rpy="0 0 3.14159265358979"/>
   </joint>
   <xacro:mujoco_ros2_control_config

File: workspace/src/robot_description/urdf/mujoco_config.xacro (robot description, xacro)
@@ -9,5 +9,5 @@
       <hardware>
         <plugin>mujoco_ros2_control/MujocoSystemInterface</plugin>
-        <param name="mujoco_model">/config/workspace/src/robot_description/mjcf/scene.xml</param>
+        <param name="mujoco_model">/config/workspace/mujoco_model/scene.xml</param>
         <param name="sim_speed_factor">0.5</param>
         <param name="headless">true</param>
@@ -15,4 +15,5 @@
         <param name="physics_sync_safety_interval">0</param>
         <param name="extra_wait_time">4</param>
+        <param name="required_active_controllers">joint_state_broadcaster,imu_sensor_broadcaster,mecanum_drive_controller,arm_trajectory_controller,gripper_controller</param>
         <!-- All MuJoCo camera streams are rendered and published at this rate. -->
         <param name="camera_publish_rate">1.0</param>
@@ -60,6 +61,6 @@
       <joint name="arm_elbow_joint">
         <command_interface name="position">
-          <param name="min">-3.141592653589793</param>
-          <param name="max">3.141592653589793</param>
+          <param name="min">-6.28318530717958</param>
+          <param name="max">6.28318530717958</param>
         </command_interface>
         <state_interface name="position"/>

Commit message: added GPD

File: workspace/src/robot_description/urdf/full_robot.xacro (robot description, xacro)
@@ -63,11 +63,42 @@
   </joint>
   <!-- ROS optical frame matching robot.xml's forward-facing camera:
-       +X right, +Y down, and +Z forward along the chassis +X axis. -->
+       +X right, +Y down, and +Z forward, tilted 30 deg downward from the
+       chassis +X axis (rotation about the chassis +Y axis). -->
   <link name="front_camera_frame"/>
   <joint name="front_camera_joint" type="fixed">
     <parent link="base_link"/>
     <child link="front_camera_frame"/>
-    <origin xyz="0.51 0 0.48"
-            rpy="-1.57079632679 0 -1.57079632679"/>
+    <origin xyz="0.5 0 0.64"
+            rpy="-2.09439510239 0 -1.57079632679"/>
+  </joint>
+  <!-- The left-facing camera trio (robot.xml: left_camera /
+       left_front_camera / left_back_camera), sitting on the chassis +Y edge
+       at y = 0.4 and at front_camera_frame's height. All three keep that
+       30 deg downward tilt (the -2.0944 roll) but point along the chassis
+       +Y axis instead of +X, which in this rpy convention is a zero yaw.
+       left_front_camera_frame and left_back_camera_frame are 0.3 m fore and
+       aft of left_camera_frame and are yawed 30 deg (pi/6) back towards it.
+       The grasp pose provider merges all three clouds into left_camera_frame
+       using these transforms, so they must stay in sync with robot.xml. -->
+  <link name="left_camera_frame"/>
+  <joint name="left_camera_joint" type="fixed">
+    <parent link="base_link"/>
+    <child link="left_camera_frame"/>
+    <origin xyz="0 0.4 0.64"
+            rpy="-2.09439510239 0 0"/>
+  </joint>
+  <link name="left_front_camera_frame"/>
+  <joint name="left_front_camera_joint" type="fixed">
+    <parent link="base_link"/>
+    <child link="left_front_camera_frame"/>
+    <origin xyz="0.3 0.4 0.64"
+            rpy="-2.09439510239 0 0.52359877560"/>
+  </joint>
+  <link name="left_back_camera_frame"/>
+  <joint name="left_back_camera_joint" type="fixed">
+    <parent link="base_link"/>
+    <child link="left_back_camera_frame"/>
+    <origin xyz="-0.3 0.4 0.64"
+            rpy="-2.09439510239 0 -0.52359877560"/>
   </joint>
   <!-- Match the MuJoCo chassis frame exactly: +X is front and +Y is left. -->

File: workspace/src/robot_description/urdf/mujoco_config.xacro (robot description, xacro)
@@ -125,4 +125,19 @@
         <param name="pointcloud_topic">/front_camera/points</param>
       </sensor>
+      <!-- The left-facing MuJoCo camera trio (robot.xml: left_camera /
+           left_front_camera / left_back_camera). The grasp pose provider
+           merges all three of these clouds into left_camera_frame. -->
+      <sensor name="left_camera">
+        <param name="frame_name">left_camera_frame</param>
+        <param name="pointcloud_topic">/left_camera/points</param>
+      </sensor>
+      <sensor name="left_front_camera">
+        <param name="frame_name">left_front_camera_frame</param>
+        <param name="pointcloud_topic">/left_front_camera/points</param>
+      </sensor>
+      <sensor name="left_back_camera">
+        <param name="frame_name">left_back_camera_frame</param>
+        <param name="pointcloud_topic">/left_back_camera/points</param>
+      </sensor>
     </ros2_control>
   </xacro:macro>

Commit message: made mujoco_ros2_control more tidy

File: workspace/src/robot_description/urdf/full_robot.xacro (robot description, xacro)
@@ -134,7 +134,4 @@
     <origin xyz="0 0 0.45" rpy="0 0 3.14159265358979"/>
   </joint>
-  <xacro:mujoco_ros2_control_config
-    write_frequency="$(arg write_frequency)"
-    physics_sync_safety_interval="$(arg physics_sync_safety_interval)"
-    extra_wait_time="$(arg extra_wait_time)"/>
+  <xacro:mujoco_ros2_control_config/>
 </robot>

File: workspace/src/robot_description/urdf/mujoco_config.xacro (robot description, xacro)
@@ -1,15 +1,9 @@
 <?xml version="1.0"?>
 <robot xmlns:xacro="http://www.ros.org/wiki/xacro">
-  <xacro:arg name="write_frequency" default="100"/>
-  <xacro:arg name="physics_sync_safety_interval" default="0.002"/>
-  <xacro:arg name="extra_wait_time" default="0"/>
-  <xacro:macro name="mujoco_ros2_control_config"
-               params="write_frequency physics_sync_safety_interval extra_wait_time">
+  <xacro:macro name="mujoco_ros2_control_config">
     <ros2_control name="MujocoSystem" type="system">
       <hardware>
         <plugin>mujoco_ros2_control/MujocoSystemInterface</plugin>
         <param name="mujoco_model">/config/workspace/mujoco_model/scene.xml</param>
-        <param name="sim_speed_factor">0.5</param>
-        <param name="headless">true</param>
         <param name="write_frequency">100</param>
         <param name="physics_sync_safety_interval">0</param>
