Commit message: added moveit setup and arm_behavior package

File: workspace/src/robot_description/urdf/arm.xacro (robot description, xacro)
@@ -18,3 +18,20 @@
     <origin xyz="0 0 0" rpy="0 0 0"/>
   </xacro:ur_robot>
+  <!-- TCP frame attached to the gripper base. Adjust this fixed transform
+       to locate the desired task point without moving the gripper itself. -->
+  <link name="arm_tcp">
+    <visual>
+      <geometry>
+        <box size="0.02 0.02 0.02"/>
+      </geometry>
+      <material name="tcp_marker">
+        <color rgba="1 0 0 1"/>
+      </material>
+    </visual>
+  </link>
+  <joint name="robotiq_85_base_to_tcp" type="fixed">
+    <parent link="robotiq_85_base_link"/>
+    <child link="arm_tcp"/>
+    <origin xyz="0 0 0.1355" rpy="0 0 0"/>
+  </joint>
 </robot>

File: workspace/src/robot_description/urdf/arm_with_gripper.xacro (robot description, xacro)
@@ -6,5 +6,5 @@
   <xacro:include filename="$(find robot_description)/urdf/gripper/gripper.xacro"/>
   <xacro:robotiq_85_gripper/>
-  <!-- Attach the gripper base to the UR5e tool frame -->
+  <!-- Attach the gripper base to the UR5e tool frame. -->
   <joint name="tool0_to_robotiq_85_base" type="fixed">
     <parent link="arm_tool0"/>

File: workspace/src/robot_description/urdf/mujoco_config.xacro (robot description, xacro)
@@ -14,5 +14,5 @@
         <param name="write_frequency">100</param>
         <param name="physics_sync_safety_interval">0</param>
-        <param name="extra_wait_time">1</param>
+        <param name="extra_wait_time">4</param>
         <!-- All MuJoCo camera streams are rendered and published at this rate. -->
         <param name="camera_publish_rate">1.0</param>

Commit message: added base locking plugin and changed gripper

File: workspace/src/robot_description/urdf/arm.xacro (robot description, xacro)
@@ -19,5 +19,7 @@
   </xacro:ur_robot>
   <!-- TCP frame attached to the gripper base. Adjust this fixed transform
-       to locate the desired task point without moving the gripper itself. -->
+       to locate the desired task point without moving the gripper itself.
+       z = 0.045 puts it at the centre of the jaw plates, which span
+       z in [0.02, 0.07] of gripper_base_link. -->
   <link name="arm_tcp">
     <visual>
@@ -30,8 +32,13 @@
     </visual>
   </link>
-  <joint name="robotiq_85_base_to_tcp" type="fixed">
-    <parent link="robotiq_85_base_link"/>
+  <!-- arm_tcp sits on the closing centre line at the mid-height of the jaw
+       plates: they span z = 0.02 .. 0.10 above gripper_base_link, so the TCP
+       is 0.04 m above the palm face they stand on and 0.04 m short of their
+       tips. GPD poses are converted onto this frame with
+       tcp_from_finger_base = 0.04 (grasp_config_conversion.py). -->
+  <joint name="gripper_base_to_tcp" type="fixed">
+    <parent link="gripper_base_link"/>
     <child link="arm_tcp"/>
-    <origin xyz="0 0 0.1355" rpy="0 0 0"/>
+    <origin xyz="0 0 0.06" rpy="0 0 0"/>
   </joint>
 </robot>

File: workspace/src/robot_description/urdf/arm_with_gripper.xacro (robot description, xacro)
@@ -3,11 +3,13 @@
   <!-- Include the UR5e arm xacro -->
   <xacro:include filename="$(find robot_description)/urdf/arm.xacro"/>
-  <!-- Include the Robotiq 2F-85 gripper xacro -->
+  <!-- Include the custom parallel-jaw gripper xacro -->
   <xacro:include filename="$(find robot_description)/urdf/gripper/gripper.xacro"/>
-  <xacro:robotiq_85_gripper/>
-  <!-- Attach the gripper base to the UR5e tool frame. -->
-  <joint name="tool0_to_robotiq_85_base" type="fixed">
+  <xacro:parallel_gripper/>
+  <!-- Attach the gripper base to the UR5e tool frame. The gripper macro is
+       authored in the tool0 convention (+Z approach, +X closing), so this is
+       an identity transform. -->
+  <joint name="tool0_to_gripper_base" type="fixed">
     <parent link="arm_tool0"/>
-    <child link="robotiq_85_base_link"/>
+    <child link="gripper_base_link"/>
     <origin xyz="0 0 0" rpy="0 0 0"/>
   </joint>

File: workspace/src/robot_description/urdf/gripper/gripper.xacro (robot description, xacro)
@@ -1,519 +1,140 @@
 <?xml version="1.0"?>
 <robot xmlns:xacro="http://www.ros.org/wiki/xacro">
-  <xacro:macro name="robotiq_85_gripper" params="">
-  <link
-    name="robotiq_85_base_link">
-    <inertial>
-      <origin
-        xyz="0.00021987 -2.3546E-10 0.030163"
-        rpy="0 0 0" />
-      <mass
-        value="0.30915" />
-      <inertia
-        ixx="0.00028972"
-        ixy="-5.7879E-10"
-        ixz="-1.8543E-06"
-        iyy="0.00030737"
-        iyz="1.682E-12"
-        izz="0.00019914" />
-    </inertial>
-    <visual>
-      <origin
-        xyz="0 0 0"
-        rpy="0 0 0" />
-      <geometry>
-        <mesh
-          filename="package://robot_description/urdf/gripper/meshes/robotiq_85_base_link_fine.STL" />
-      </geometry>
-      <material
-        name="">
-        <color
-          rgba="0.1 0.1 0.1 1" />
-      </material>
-    </visual>
-    <collision>
-      <origin
-        xyz="0 0 0"
-        rpy="0 0 0" />
-      <geometry>
-        <mesh
-          filename="package://robot_description/urdf/gripper/meshes/robotiq_85_base_link_coarse.STL" />
-      </geometry>
-    </collision>
-  </link>
-  <link
-    name="left_outer_knuckle">
-    <inertial>
-      <origin
-        xyz="0.0178331863169983 3.68915177224286E-11 0.0021442477325704"
-        rpy="0 0 0" />
-      <mass
-        value="0.00684838849434396" />
-      <inertia
-        ixx="2.66832029033166E-07"
-        ixy="1.66142314639824E-15"
-        ixz="1.45945633322873E-07"
-        iyy="1.3889233257419E-06"
-        iyz="2.82951161241588E-15"
-        izz="1.26603336914415E-06" />
-    </inertial>
-    <visual>
-      <origin
-        xyz="0 0 0"
-        rpy="0 0 0" />
-      <geometry>
-        <mesh
-          filename="package://robot_description/urdf/gripper/meshes/outer_knuckle_fine.STL" />
-      </geometry>
-      <material
-        name="">
-        <color
-          rgba="0.1 0.1 0.1 1" />
-      </material>
-    </visual>
-    <collision>
-      <origin
-        xyz="0 0 0"
-        rpy="0 0 0" />
-      <geometry>
-        <mesh
-          filename="package://robot_description/urdf/gripper/meshes/outer_knuckle_coarse.STL" />
-      </geometry>
-    </collision>
-  </link>
-  <joint
-    name="finger_joint"
-    type="revolute">
-    <origin
-      xyz="0.0306011444260539 0 0.0627920162695395"
-      rpy="0 0 0" />
-    <parent
-      link="robotiq_85_base_link" />
-    <child
-      link="left_outer_knuckle" />
-    <axis
-      xyz="0 -1 0" />
-    <limit
-	  lower="0"
-      upper="0.725"
-      velocity="2.0"
-      effort="10000" />
-  </joint>
-  <link
-    name="left_outer_finger">
-    <inertial>
-      <origin
-        xyz="0.00131451599174296 2.88942057994543E-15 0.0215404163180413"
-        rpy="0 0 0" />
-      <mass
-        value="0.0273093985570947" />
-      <inertia
-        ixx="8.51629628283022E-06"
-        ixy="2.58174336207405E-19"
-        ixz="3.83829504344079E-07"
-        iyy="6.9133328065108E-06"
-        iyz="-7.58589926143789E-19"
-        izz="2.25006832221981E-06" />
-    </inertial>
-    <visual>
-      <origin
-        xyz="0 0 0"
-        rpy="0 0 0" />
-      <geometry>
-        <mesh
-          filename="package://robot_description/urdf/gripper/meshes/outer_finger_fine.STL" />
-      </geometry>
-      <material
-        name="">
-        <color
-          rgba="0.1 0.1 0.1 1" />
-      </material>
-    </visual>
-    <collision>
-      <origin
-        xyz="0 0 0"
-        rpy="0 0 0" />
-      <geometry>
-        <mesh
-          filename="package://robot_description/urdf/gripper/meshes/outer_finger_coarse.STL" />
-      </geometry>
-    </collision>
-  </link>
-  <joint
-    name="left_outer_finger_joint"
-    type="fixed">
-    <origin
-      xyz="0.0316910442266543 0 -0.00193396375724605"
-      rpy="0 0 0" />
-    <parent
-      link="left_outer_knuckle" />
-    <child
-      link="left_outer_finger" />
-    <axis
-      xyz="0 -1 0" />
-  </joint>
-  <link
-    name="left_inner_knuckle">
-    <inertial>
-      <origin
-        xyz="0.017097546626628 -3.93808524389535E-10 0.0224918438201868"
-        rpy="0 0 0" />
-      <mass
-        value="0.0110930853895903" />
-      <inertia
-        ixx="4.23392770691541E-06"
-        ixy="5.748978936968E-15"
-        ixz="1.78855677119788E-06"
-        iyy="3.96548790524392E-06"
-        iyz="1.05464666369669E-14"
-        izz="3.24068002883007E-06" />
-    </inertial>
-    <visual>
-      <origin
-        xyz="0 0 0"
-        rpy="0 0 0" />
-      <geometry>
-        <mesh
-          filename="package://robot_description/urdf/gripper/meshes/inner_knuckle_fine.STL" />
-      </geometry>
-      <material
-        name="">
-        <color
-          rgba="0.1 0.1 0.1 1" />
-      </material>
-    </visual>
-    <collision>
-      <origin
-        xyz="0 0 0"
-        rpy="0 0 0" />
-      <geometry>
-        <mesh
-          filename="package://robot_description/urdf/gripper/meshes/inner_knuckle_coarse.STL" />
-      </geometry>
-    </collision>
-  </link>
-  <joint
-    name="left_inner_knuckle_joint"
-    type="revolute">
-    <origin
-      xyz="0.0127000000001501 0 0.0693074999999639"
-      rpy="0 0 0" />
-    <parent
-      link="robotiq_85_base_link" />
-    <child
-      link="left_inner_knuckle" />
-    <axis
-      xyz="0 -1 0" />
-    <limit
-      lower="0"
-      upper="0.8757"
-      velocity="2.0"
-      effort="10000" />
-    <mimic
-      joint="finger_joint"
-      multiplier="1"
-      offset="0" />
-  </joint>
-  <link
-    name="left_inner_finger">
-    <inertial>
-      <origin
-        xyz="0.0060275613594574 -6.29183141465421E-15 0.00669925693133241"
-        rpy="0 0 0" />
-      <mass
-        value="0.00724255346165745" />
-      <inertia
-        ixx="1.47824274053603E-06"
-        ixy="-3.94884463570303E-19"
-        ixz="-3.45268847648622E-07"
-        iyy="1.70064480838395E-06"
-        iyz="3.5059838910097E-19"
-        izz="4.77151336838364E-07" />
-    </inertial>
-    <visual>
-      <origin
-        xyz="0 0 0"
-        rpy="0 0 0" />
-      <geometry>
-        <mesh
-          filename="package://robot_description/urdf/gripper/meshes/inner_finger_fine.STL" />
-      </geometry>
-      <material
-        name="">
-        <color
-          rgba="0.1 0.1 0.1 1" />
-      </material>
-    </visual>
-    <collision>
-      <origin
-        xyz="0 0 0"
-        rpy="0 0 0" />
-      <geometry>
-        <mesh
-          filename="package://robot_description/urdf/gripper/meshes/inner_finger_coarse.STL" />
-      </geometry>
-    </collision>
-  </link>
-  <joint
-    name="left_inner_finger_joint"
-    type="revolute">
-    <origin
-      xyz="0.034585310861294 0 0.0454970193817975"
-      rpy="0 0 0" />
-    <parent
-      link="left_inner_knuckle" />
-    <child
-      link="left_inner_finger" />
-    <axis
-      xyz="0 -1 0" />
-    <limit
-      lower="0"
-      upper="0.8757"
-      velocity="2.0"
-      effort="10000" />
-    <mimic
-      joint="finger_joint"
-      multiplier="-1"
-      offset="0" />
-  </joint>
-  <link
-    name="right_inner_knuckle">
-    <inertial>
-      <origin
-        xyz="0.0168606186773776 3.93808471820465E-10 0.0226699950793434"
-        rpy="0 0 0" />
-      <mass
-        value="0.0110930853895903" />
-      <inertia
-        ixx="4.27134775939882E-06"
-        ixy="-8.53568456728898E-15"
-        ixz="1.77774229944246E-06"
-        iyy="3.96548790524392E-06"
-        iyz="-8.45108024914164E-15"
-        izz="3.20325997634666E-06" />
-    </inertial>
-    <visual>
-      <origin
-        xyz="0 0 0"
-        rpy="0 0 0" />
-      <geometry>
-        <mesh
-          filename="package://robot_description/urdf/gripper/meshes/inner_knuckle_fine.STL" />
-      </geometry>
-      <material
-        name="">
-        <color
-          rgba="0.1 0.1 0.1 1" />
-      </material>
-    </visual>
-    <collision>
-      <origin
-        xyz="0 0 0"
-        rpy="0 0 0" />
-      <geometry>
-        <mesh
-          filename="package://robot_description/urdf/gripper/meshes/inner_knuckle_coarse.STL" />
-      </geometry>
-    </collision>
-  </link>
-  <joint
-    name="right_inner_knuckle_joint"
-    type="revolute">
-    <origin
-      xyz="-0.0126999999998499 0 0.0693075000000361"
-      rpy="0 0 3.14159265358979" />
-    <parent
-      link="robotiq_85_base_link" />
-    <child
-      link="right_inner_knuckle" />
-    <axis
-      xyz="0 1 0" />
-    <limit
-      lower="0"
-      upper="0.8757"
-      velocity="2.0"
-      effort="10000" />
-    <mimic
-      joint="finger_joint"
-      multiplier="-1"
-      offset="0" />
-  </joint>
-  <link
-    name="right_inner_finger">
-    <inertial>
-      <origin
-        xyz="0.00602756228812038 -6.47284509480176E-15 0.00669925609578108"
-        rpy="0 0 0" />
-      <mass
-        value="0.00724255346165744" />
-      <inertia
-        ixx="1.47824283625957E-06"
-        ixy="-3.95952064019123E-19"
-        ixz="-3.45268708875543E-07"
-        iyy="1.70064480838394E-06"
-        iyz="3.55286507960029E-19"
-        izz="4.77151241114822E-07" />
-    </inertial>
-    <visual>
-      <origin
-        xyz="0 0 0"
-        rpy="0 0 0" />
-      <geometry>
-        <mesh
-          filename="package://robot_description/urdf/gripper/meshes/inner_finger_fine.STL" />
-      </geometry>
-      <material
-        name="">
-        <color
-          rgba="0.1 0.1 0.1 1" />
-      </material>
-    </visual>
-    <collision>
-      <origin
-        xyz="0 0 0"
-        rpy="0 0 0" />
-      <geometry>
-        <mesh
-          filename="package://robot_description/urdf/gripper/meshes/inner_finger_coarse.STL" />
-      </geometry>
-    </collision>
-  </link>
-  <joint
-    name="right_inner_finger_joint"
-    type="revolute">
-    <origin
-      xyz="0.0341060475457406 0 0.0458573878541688"
-      rpy="0 0 0" />
-    <parent
-      link="right_inner_knuckle" />
-    <child
-      link="right_inner_finger" />
-    <axis
-      xyz="0 1 0" />
-    <limit
-      lower="0"
-      upper="0.8757"
-      velocity="2.0"
-      effort="10000" />
-    <mimic
-      joint="finger_joint"
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
File: workspace/src/robot_description/urdf/mujoco_config.xacro (robot description, xacro)
@@ -92,9 +92,13 @@
         <state_interface name="effort"/>
       </joint>
-      <!-- Gripper Joint -->
+      <!-- Gripper Joint. The prismatic jaw travel of the custom parallel
+           gripper: 0 is fully open, 0.055 has the two jaws meeting on the
+           palm centre line. Must match the finger_joint actuator ctrlrange
+           in scene.xml. right_finger_joint mimics this one, so it needs no
+           interface of its own. -->
       <joint name="finger_joint">
         <command_interface name="position">
           <param name="min">0</param>
-          <param name="max">0.725</param>
+          <param name="max">0.055</param>
         </command_interface>
         <state_interface name="position"/>
